File: ELE_PWR_SW_B1.kicad_sch (KiCad schematic)
At the start: 58 parts, among them J101 Conn_01x02_Pin, Q101 2N7002, Q102 SM4185, Q103 SM4185, Q104 SM4185, Q105 SM4185, Q106 2N7002, Q107 SM4185, Q108 SM4185

Commit message: Update readme
Other:
- company: (none) -> Les Opossums - Gabriel DE MELO SOUZA
- title: (none) -> Power Switch - Main
Changed lines of the file:
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@@
 	(generator_version "9.0")
 	(paper "A4")
+	(title_block
+		(title "Power Switch - Main")
+		(date "2025-11-15")
+		(rev "B1")
+		(company "Les Opossums - Gabriel DE MELO SOUZA")
+	)
 	(rectangle
 		(start 15.24 101.6)
